File: pcb/mcu_integration.kicad_pcb (KiCad board)
At the start: 4 copper layers, 70 x 70 mm, 81 parts, among them IC1 TL7660IDGKR, IC2 TL081IDT, IC3 LMT87DCKT, IC6 AD844_OPAMP_AL, IC7 FOD814_OPTO_AL, J1 Conn_01x05, J2 Conn_01x03, J5 DM3BT-DSF-PEJS, U1 STM32F103RBTx, U2 LTC4300A-1IMS8_PBF, U3 REF192_AL, U4 TPS79933QDDCRQ1

Commit message: Silkscreen clean up
Parts:
- moved G*** 1.09 mm to (117.9, 83.0)
Routing:
- net GND: vias 174 -> 171

Commit message: Replaced wire to board connectors with screw terminals
Parts:
- removed I2C_1: Conn_01x02, Connector_PinHeader_2.54mm:PinHeader_1x02_P2.54mm_Vertical
- removed J_AD2: Conn_01x04, Connector_PinHeader_2.54mm:PinHeader_1x04_P2.54mm_Vertical
- removed J_SIG1, PWR1: Conn_01x03, Connector_PinHeader_2.54mm:PinHeader_1x03_P2.54mm_Vertical
- added J3: 1751264, Screw Terminal 1x4:CONN_1751264_PXC, F.Cu at (146.7, 124.8)
- added J4: 1751264, Screw Terminal 1x4:CONN_1751264_PXC, F.Cu at (164.9, 124.8)
- added J6: 1751251, Screw Terminal 1x3:CONN_1751251_PXC, F.Cu at (173.3, 78.9)
- added J7: 1751251, Screw Terminal 1x3:CONN_1751251_PXC, F.Cu at (144.8, 68.6)
- R10: value 9K -> 10K
- moved G*** 12.5 mm to (160.5, 111.4)
- moved R5 3.95 mm to (161.1, 119.5), turned to -90 degrees
- moved C14 3.32 mm to (160.1, 119.5), turned to 90 degrees
- moved R6 2.80 mm to (159.1, 119.5), turned to 90 degrees
- moved C15 2.21 mm to (158.1, 119.5)
- moved R7 1.75 mm to (157.1, 119.5), turned to -90 degrees
- moved J5 1.70 mm to (160.3, 72.3)
- moved C16 1.19 mm to (156.1, 119.5), turned to 90 degrees
- moved R8 0.75 mm to (155.1, 119.5), turned to 90 degrees
- moved C27 0.73 mm to (160.1, 84.2)
- moved C33 0.73 mm to (160.1, 83.0)
Routing:
- net ADC1_IN9_LMT87: track 17.1 -> 47.0 mm, vias 0 -> 1
- net ADC1_IN6_VREF_AL: track 51.4 -> 74.8 mm
- net ADC1_IN14_OPTO_F_AL: track 40.1 -> 63.0 mm
- net ADC1_IN15_OPTO_E_AL: track 49.9 -> 72.2 mm
- net ADC1_IN3_OPAMP_AL: track 56.0 -> 70.8 mm, vias 1 -> 2
- net SIG_SQUARE: track 40.2 -> 44.7 mm
- net GND: track 27.5 -> 31.7 mm, vias 171 -> 166
- net 3.3V Output: track 53.7 -> 49.7 mm
- net Net-(C43-Pad2): track 20.4 -> 22.3 mm
- net I2C_SDA: track 16.1 -> 17.3 mm
- net I2C_SCL: track 13.2 -> 14.4 mm
- net RC_OUTPUT: track 14.0 -> 15.1 mm
- net ADC1_IN0_SINE: track 64.9 -> 66.0 mm
- net -5V Output: track 123.7 -> 122.6 mm
- net /SPI2_SCK: track 35.3 -> 36.2 mm
Other:
- board text added: "TEMP"
